Commit message: Added Gazebo configuration and launch file

File: description/robot_core.xacro (robot description, xacro)
@@ -46,4 +46,5 @@
         <origin xyz="0 0.175 0" rpy="-${pi/2} 0 0"/>
         <axis xyz="0 0 1"/>
+        <limit effort="0.05" velocity="10.0"/>
     </joint>
     <link name="left_wheel">
@@ -56,5 +57,5 @@
         <collision>
             <geometry>
-                <cylinder length="0.04" radius="0.05"/>
+                <sphere radius="0.05"/>
             </geometry>
         </collision>
@@ -69,4 +70,5 @@
         <origin xyz="0 -0.175 0" rpy="${pi/2} 0 0"/>
         <axis xyz="0 0 -1"/>
+        <limit effort="0.05" velocity="10.0"/>
     </joint>
     <link name="right_wheel">
@@ -79,5 +81,5 @@
         <collision>
             <geometry>
-                <cylinder length="0.04" radius="0.05"/>
+                <sphere radius="0.05"/>
             </geometry>
         </collision>
@@ -108,3 +110,7 @@
         </xacro:inertial_sphere>
     </link>
+    <gazebo reference="caster_wheel">
+        <mu1 value="0.0"/>
+        <mu2 value="0.0"/>
+    </gazebo>
 </robot>
